File: hardware/t1s_hat.kicad_sch (KiCad schematic)
At the start: 38 parts, among them CN1 T1S BUS P N N P, J1 2x20 socket (riser stack), U1 LAN8651, Y1 25.000MHz CL12

Commit message: Rev B review follow-ups: X7R CCOMP, probe labels, ferrite note, 23 mm
Checked against the board file and Microchip's documents:
- C4 (CCOMP) X5R -> X7R (Yageo CC0805KKX7R8BB475, C354262). The
  checklist says 'metal film', the data sheet does not; recorded.
- J1 pins 15-24 carry all six host signals plus 3V3 and GND: labelled
  on the silkscreen as the bring-up probe points.
- Ferrite beads need a local 10 uF (checklist); FB1-4 documented as
  0 ohm links, with which the single C6 is compliant.
- Stack height text corrected to the calculated ~23 mm everywhere.
- README 'Review notes': why the P N N P connector stays (the node's
  stub is 15.92 mm on both legs; the difference is the through-bus,
  ~93 ps) and why no series-R on SCLK/MOSI (driver is the ESP32).
DRC 0 errors, ERC 0 errors, mechanical 0.00000 mm.
Parts:
- C4: value 4.7uF low-ESR -> 4.7uF X7R; LCSC C1779 -> C354262
Changed lines of the file:
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@@
       (effects (font (size 1.27 1.27)) hide)
     )
-    (property "Description" "VDDA supply island option: 0 ohm fitted; may be replaced by a ~300 ohm @ 100 MHz bead (e.g. Wuerth 742792640)." (at 157.48 44.45 0)
+    (property "Description" "VDDA supply island option: 0 ohm fitted. A real bead needs a local 10 uF after it (DS60001746D); may be replaced by a ~300 ohm @ 100 MHz bead (e.g. Wuerth 742792640)." (at 157.48 44.45 0)
       (effects (font (size 1.27 1.27)) hide)
     )
@@
       (effects (font (size 1.27 1.27)) hide)
     )
-    (property "Description" "VDDAU supply island option: 0 ohm fitted." (at 222.25 44.45 0)
+    (property "Description" "VDDAU supply island option: 0 ohm fitted. A real bead needs a local 10 uF after it (DS60001746D)." (at 222.25 44.45 0)
       (effects (font (size 1.27 1.27)) hide)
     )
@@
       (effects (font (size 1.27 1.27)) hide)
     )
-    (property "Description" "VDDP (pin 7) supply island option: 0 ohm fitted." (at 62.23 44.45 0)
+    (property "Description" "VDDP (pin 7) supply island option: 0 ohm fitted. A real bead needs a local 10 uF after it (DS60001746D)." (at 62.23 44.45 0)
       (effects (font (size 1.27 1.27)) hide)
     )
@@
       (effects (font (size 1.27 1.27)) hide)
     )
-    (property "Description" "VDDP (pin 17) supply island option: 0 ohm fitted." (at 110.49 80.01 0)
+    (property "Description" "VDDP (pin 17) supply island option: 0 ohm fitted. A real bead needs a local 10 uF after it (DS60001746D)." (at 110.49 80.01 0)
       (effects (font (size 1.27 1.27)) hide)
     )
@@
       (effects (font (size 1.27 1.27)) (justify left))
     )
-    (property "Value" "4.7uF low-ESR" (at 291.76 45.05 0)
+    (property "Value" "4.7uF X7R" (at 291.76 45.05 0)
       (effects (font (size 1.27 1.27)) (justify left))
     )
@@
       (effects (font (size 1.27 1.27)) hide)
     )
-    (property "Description" "CCOMP: internal +1.8 V core LDO compensation. REQUIRED, low ESR, to the ground plane (LAN8651 only)." (at 289.56 44.45 0)
-      (effects (font (size 1.27 1.27)) hide)
-    )
-    (property "LCSC" "C1779" (at 289.56 44.45 0)
-      (effects (font (size 1.27 1.27)) hide)
-    )
+    (property "Description" "CCOMP: internal +1.8 V core LDO compensation. REQUIRED, low ESR, to the ground plane (LAN8651 only). X7R MLCC; see ELECTRICAL.md on the checklist's 'metal film' wording." (at 289.56 44.45 0)
+      (effects (font (size 1.27 1.27)) hide)
+    )
+    (property "LCSC" "C354262" (at 289.56 44.45 0)
+      (effects (font (size 1.27 1.27)) hide)
+    )
